File: DimmerWifi.kicad_pcb (KiCad board)
At the start: 2 copper layers, 13 parts, among them J1 AC, J2 Load, J3 Conn_01x04, U1 MOC3021M, U2 4N25

Commit message: fix
Parts:
- removed D1: Q_TRIAC_AAG, TO_SOT_Packages_THT:TO-220-3_Vertical
- removed D3: LED, LEDs:LED_D5.0mm
- added Q1: TRIAC_BTA, w_to:to220, F.Cu at (176.3, 77.0)
- J1, J2: footprint TerminalBlocks_Phoenix:TerminalBlock_Phoenix_MPT-2.54mm_2pol -> w_conn_mkds:mkds_1,5-2
- J3: footprint Pin_Headers:Pin_Header_Angled_1x04_Pitch2.54mm -> w_pin_strip:pin_strip_2mm_4
- R1, R2, R3, R4, R5: footprint Resistors_THT:R_Axial_DIN0411_L9.9mm_D3.6mm_P7.62mm_Vertical -> w_pth_resistors:RC03
- moved J3 68.5 mm to (199.4, 76.7), turned to 270 degrees
- moved R5 61.9 mm to (195.6, 67.3), turned to 90 degrees
- moved R4 46.2 mm to (194.3, 83.3), turned to 0 degrees
- moved U2 43.3 mm to (184.7, 63.5), turned to 0 degrees
- moved U1 42.4 mm to (194.6, 79.5), turned to 180 degrees
- moved D2 36.9 mm to (180.8, 63.8), turned to 270 degrees
- moved R1 33.8 mm to (183.9, 75.2), turned to 270 degrees
- moved J2 28.9 mm to (165.6, 67.8)
- moved J1 28.8 mm to (165.6, 78.2)
- moved R2 23.1 mm to (172.2, 71.1), turned to 270 degrees
- moved R3 17.2 mm to (180.8, 77.0), turned to 270 degrees
Connections:
- J3 pad 4: Net-(D3-Pad2) -> Net-(J3-Pad4)
- R4 pad 2: Net-(D3-Pad1) -> Net-(J3-Pad4)
Routing:
- net Net-(Q1-Pad1): track 0.00 -> 25.1 mm
- net Net-(J3-Pad2): track 0.00 -> 21.4 mm
- net /Fase: track 0.00 -> 20.7 mm
- net Net-(J2-Pad1): track 0.00 -> 18.6 mm
- net GND: track 0.00 -> 16.5 mm
- net /Neutro: track 0.00 -> 12.4 mm
- net Net-(D2-Pad3): track 0.00 -> 10.0 mm
- net Net-(R3-Pad2): track 0.00 -> 7.79 mm
- net Net-(R4-Pad1): track 0.00 -> 6.68 mm
- net +3V3: track 0.00 -> 5.80 mm
- net Net-(D2-Pad2): track 0.00 -> 5.03 mm
- net Net-(J3-Pad4): track 0.00 -> 4.13 mm
- net Net-(D2-Pad4): track 0.00 -> 4.10 mm
- net Net-(D2-Pad1): track 0.00 -> 3.92 mm
- net (no net): track 0.00 -> 0.97 mm
Other:
- board outline added: 40.1 x 23.6 mm
- rule pad_to_mask_clearance: 0.2 -> 0

Commit message: add esp32
Parts:
- added U3: ESP32-WROOM, ESP32-footprints-Lib:ESP32-WROOM, F.Cu at (182.9, 94.0)
Connections:
- net +3V3 renamed +3.3V
Other:
- board outline removed
